Commit message: add g1 simplified urdf

File: source/locolab/locolab/assets/robots/unitree/G1/urdf/g1_description/g1_29dof_torsobase_cylinder.urdf (robot description, URDF)
Before this commit: robot g1_29dof_lock_waist, 40 links, 39 joints
Links:
- removed link d435_link
- removed link imu_in_pelvis
- removed link imu_in_torso
- removed link mid360_link
- added link imu_link
- link head_link: geometry collision sphere radius=0.07; visual mesh filename=../meshes/head_link.STL
- link left_ankle_pitch_link: geometry visual mesh filename=../meshes/left_ankle_pitch_link.STL
- link left_ankle_roll_link: geometry collision box size=0.18 0.046 0.03; collision cylinder length=0.046 radius=0.015
- link left_elbow_link: geometry collision cylinder length=0.12 radius=0.036; visual mesh filename=../meshes/left_elbow_link.STL
- link left_hip_pitch_link: geometry collision cylinder length=0.1 radius=0.048; visual mesh filename=../meshes/left_hip_pitch_link.STL
- link left_hip_roll_link: geometry visual mesh filename=../meshes/left_hip_roll_link.STL
- link left_hip_yaw_link: geometry collision cylinder length=0.16 radius=0.055; visual mesh filename=../meshes/left_hip_yaw_link.STL
- link left_knee_link: geometry collision box size=0.06 0.04 0.12; collision box size=0.1 0.075 0.2
- link left_rubber_hand: geometry collision box size=0.12 0.03 0.08; visual mesh filename=../meshes/left_rubber_hand.STL
- link left_shoulder_pitch_link: geometry collision cylinder length=0.07 radius=0.036; visual mesh filename=../meshes/left_shoulder_pitch_link.STL
- link left_shoulder_roll_link: geometry visual mesh filename=../meshes/left_shoulder_roll_link.STL
- link left_shoulder_yaw_link: geometry collision cylinder length=0.07 radius=0.036; collision cylinder length=0.076 radius=0.036
- link left_wrist_pitch_link: geometry visual mesh filename=../meshes/left_wrist_pitch_link.STL
- link left_wrist_roll_link: geometry visual mesh filename=../meshes/left_wrist_roll_link.STL
- link left_wrist_yaw_link: geometry visual mesh filename=../meshes/left_wrist_yaw_link.STL
- link logo_link: geometry visual mesh filename=../meshes/logo_link.STL
- link pelvis: geometry collision cylinder length=0.12 radius=0.06; visual mesh filename=../meshes/pelvis.STL
- link pelvis_contour_link: geometry visual mesh filename=../meshes/pelvis_contour_link.STL
- link right_ankle_pitch_link: geometry visual mesh filename=../meshes/right_ankle_pitch_link.STL
- link right_ankle_roll_link: geometry collision box size=0.18 0.046 0.03; collision cylinder length=0.046 radius=0.015
- link right_elbow_link: geometry collision cylinder length=0.12 radius=0.036; visual mesh filename=../meshes/right_elbow_link.STL
- link right_hip_pitch_link: geometry collision cylinder length=0.1 radius=0.048; visual mesh filename=../meshes/right_hip_pitch_link.STL
- link right_hip_roll_link: geometry visual mesh filename=../meshes/right_hip_roll_link.STL
- link right_hip_yaw_link: geometry collision cylinder length=0.16 radius=0.055; visual mesh filename=../meshes/right_hip_yaw_link.STL
- link right_knee_link: geometry collision box size=0.06 0.03 0.12; collision box size=0.09 0.075 0.2
- link right_rubber_hand: geometry collision box size=0.12 0.03 0.08; visual mesh filename=../meshes/right_rubber_hand.STL
- link right_shoulder_pitch_link: geometry collision cylinder length=0.07 radius=0.036; visual mesh filename=../meshes/right_shoulder_pitch_link.STL
- link right_shoulder_roll_link: geometry visual mesh filename=../meshes/right_shoulder_roll_link.STL
- link right_shoulder_yaw_link: geometry collision cylinder length=0.07 radius=0.036; collision cylinder length=0.076 radius=0.036
- link right_wrist_pitch_link: geometry visual mesh filename=../meshes/right_wrist_pitch_link.STL
- link right_wrist_roll_link: geometry visual mesh filename=../meshes/right_wrist_roll_link.STL
- link right_wrist_yaw_link: geometry visual mesh filename=../meshes/right_wrist_yaw_link.STL
- link torso_link: geometry collision box size=0.1 0.196 0.24; collision box size=0.12 0.12 0.34
- link waist_roll_link: geometry visual mesh filename=../meshes/waist_roll_link.STL
- link waist_support_link: geometry visual mesh filename=../meshes/waist_support_link.STL
- link waist_yaw_link: geometry visual mesh filename=../meshes/waist_yaw_link.STL
Joints:
- removed joint d435_joint
- removed joint imu_in_pelvis_joint
- removed joint imu_in_torso_joint
- removed joint mid360_joint
- added joint imu_joint: type fixed, parent torso_link, child imu_link, origin xyz=-0.03959 -0.00224 0.13792 rpy=0 0 0
- joint left_ankle_pitch_joint: limit lower=-0.87267 upper=0.5236 effort=35 velocity=30 -> lower=-0.87267 upper=0.5236 effort=50 velocity=37
- joint left_ankle_roll_joint: limit lower=-0.2618 upper=0.2618 effort=35 velocity=30 -> lower=-0.2618 upper=0.2618 effort=50 velocity=37
- joint right_ankle_pitch_joint: limit lower=-0.87267 upper=0.5236 effort=35 velocity=30 -> lower=-0.87267 upper=0.5236 effort=50 velocity=37
- joint right_ankle_roll_joint: limit lower=-0.2618 upper=0.2618 effort=35 velocity=30 -> lower=-0.2618 upper=0.2618 effort=50 velocity=37
- joint waist_pitch_joint: child torso_link -> waist_roll_link; limit lower=-0.52 upper=0.52 effort=35 velocity=30 -> lower=-0.52 upper=0.52 effort=50 velocity=37; origin xyz=0 0 0.019 rpy=0 0 0 -> xyz=0 0 -0.019 rpy=0 0 0; parent waist_roll_link -> torso_link; type fixed -> revolute
- joint waist_roll_joint: child waist_roll_link -> waist_yaw_link; limit lower=-0.52 upper=0.52 effort=35 velocity=30 -> lower=-0.52 upper=0.52 effort=50 velocity=37; origin xyz=-0.0039635 0 0.035 rpy=0 0 0 -> xyz=0.0039635 0 -0.035 rpy=0 0 0; parent waist_yaw_link -> waist_roll_link; type fixed -> revolute
- joint waist_yaw_joint: child waist_yaw_link -> pelvis; parent pelvis -> waist_yaw_link

File: source/locolab/locolab/assets/robots/unitree/G1/urdf/g1_description/g1_29dof_torsobase_simplified.urdf (robot description, URDF)
Before this commit: robot g1_29dof_lock_waist, 40 links, 39 joints
Links:
- removed link d435_link
- removed link imu_in_pelvis
- removed link imu_in_torso
- removed link mid360_link
- added link imu_link
- link head_link: geometry collision sphere radius=0.07; visual mesh filename=meshes/head_link.STL
- link left_ankle_pitch_link: geometry visual mesh filename=meshes/left_ankle_pitch_link.STL
- link left_ankle_roll_link: geometry collision cylinder length=0.05 radius=0.01; collision cylinder length=0.05 radius=0.01
- link left_elbow_link: geometry collision cylinder length=0.12 radius=0.036; visual mesh filename=meshes/left_elbow_link.STL
- link left_hip_pitch_link: geometry collision cylinder length=0.1 radius=0.048; visual mesh filename=meshes/left_hip_pitch_link.STL
- link left_hip_roll_link: geometry visual mesh filename=meshes/left_hip_roll_link.STL
- link left_hip_yaw_link: geometry collision cylinder length=0.16 radius=0.055; visual mesh filename=meshes/left_hip_yaw_link.STL
- link left_knee_link: geometry collision box size=0.06 0.04 0.12; collision box size=0.1 0.075 0.2
- link left_rubber_hand: geometry collision box size=0.12 0.03 0.08; visual mesh filename=meshes/left_rubber_hand.STL
- link left_shoulder_pitch_link: geometry collision cylinder length=0.07 radius=0.036; visual mesh filename=meshes/left_shoulder_pitch_link.STL
- link left_shoulder_roll_link: geometry visual mesh filename=meshes/left_shoulder_roll_link.STL
- link left_shoulder_yaw_link: geometry collision cylinder length=0.07 radius=0.036; collision cylinder length=0.076 radius=0.036
- link left_wrist_pitch_link: geometry visual mesh filename=meshes/left_wrist_pitch_link.STL
- link left_wrist_roll_link: geometry visual mesh filename=meshes/left_wrist_roll_link.STL
- link left_wrist_yaw_link: geometry visual mesh filename=meshes/left_wrist_yaw_link.STL
- link logo_link: geometry visual mesh filename=meshes/logo_link.STL
- link pelvis: geometry collision cylinder length=0.12 radius=0.06; visual mesh filename=meshes/pelvis.STL
- link pelvis_contour_link: geometry visual mesh filename=meshes/pelvis_contour_link.STL
- link right_ankle_pitch_link: geometry visual mesh filename=meshes/right_ankle_pitch_link.STL
- link right_ankle_roll_link: geometry collision cylinder length=0.05 radius=0.01; collision cylinder length=0.05 radius=0.01
- link right_elbow_link: geometry collision cylinder length=0.12 radius=0.036; visual mesh filename=meshes/right_elbow_link.STL
- link right_hip_pitch_link: geometry collision cylinder length=0.1 radius=0.048; visual mesh filename=meshes/right_hip_pitch_link.STL
- link right_hip_roll_link: geometry visual mesh filename=meshes/right_hip_roll_link.STL
- link right_hip_yaw_link: geometry collision cylinder length=0.16 radius=0.055; visual mesh filename=meshes/right_hip_yaw_link.STL
- link right_knee_link: geometry collision box size=0.06 0.03 0.12; collision box size=0.09 0.075 0.2
- link right_rubber_hand: geometry collision box size=0.12 0.03 0.08; visual mesh filename=meshes/right_rubber_hand.STL
- link right_shoulder_pitch_link: geometry collision cylinder length=0.07 radius=0.036; visual mesh filename=meshes/right_shoulder_pitch_link.STL
- link right_shoulder_roll_link: geometry visual mesh filename=meshes/right_shoulder_roll_link.STL
- link right_shoulder_yaw_link: geometry collision cylinder length=0.07 radius=0.036; collision cylinder length=0.076 radius=0.036
- link right_wrist_pitch_link: geometry visual mesh filename=meshes/right_wrist_pitch_link.STL
- link right_wrist_roll_link: geometry visual mesh filename=meshes/right_wrist_roll_link.STL
- link right_wrist_yaw_link: geometry visual mesh filename=meshes/right_wrist_yaw_link.STL
- link torso_link: geometry collision box size=0.1 0.196 0.24; collision box size=0.12 0.12 0.34
- link waist_support_link: geometry visual mesh filename=meshes/waist_support_link.STL
Joints:
- removed joint d435_joint
- removed joint imu_in_pelvis_joint
- removed joint imu_in_torso_joint
- removed joint mid360_joint
- added joint imu_joint: type fixed, parent torso_link, child imu_link, origin xyz=-0.03959 -0.00224 0.13792 rpy=0 0 0
- joint left_ankle_pitch_joint: limit lower=-0.87267 upper=0.5236 effort=35 velocity=30 -> lower=-0.87267 upper=0.5236 effort=50 velocity=37
- joint left_ankle_roll_joint: limit lower=-0.2618 upper=0.2618 effort=35 velocity=30 -> lower=-0.2618 upper=0.2618 effort=50 velocity=37
- joint right_ankle_pitch_joint: limit lower=-0.87267 upper=0.5236 effort=35 velocity=30 -> lower=-0.87267 upper=0.5236 effort=50 velocity=37
- joint right_ankle_roll_joint: limit lower=-0.2618 upper=0.2618 effort=35 velocity=30 -> lower=-0.2618 upper=0.2618 effort=50 velocity=37
- joint waist_pitch_joint: child torso_link -> waist_roll_link; limit lower=-0.52 upper=0.52 effort=35 velocity=30 -> lower=-0.52 upper=0.52 effort=50 velocity=37; origin xyz=0 0 0.019 rpy=0 0 0 -> xyz=0 0 -0.019 rpy=0 0 0; parent waist_roll_link -> torso_link; type fixed -> revolute
- joint waist_roll_joint: child waist_roll_link -> waist_yaw_link; limit lower=-0.52 upper=0.52 effort=35 velocity=30 -> lower=-0.52 upper=0.52 effort=50 velocity=37; origin xyz=-0.0039635 0 0.035 rpy=0 0 0 -> xyz=0.0039635 0 -0.035 rpy=0 0 0; parent waist_yaw_link -> waist_roll_link; type fixed -> revolute
- joint waist_yaw_joint: child waist_yaw_link -> pelvis; parent pelvis -> waist_yaw_link
