Commit message: update tasks

File: source/locolab/locolab/assets/robots/unitree/G1/urdf/g1_description/g1_29dof_beyondmimic_torso_base.urdf (robot description, URDF)
Before this commit: robot g1, 40 links, 39 joints
Joints:
- joint waist_pitch_joint: axis 0 1 0 -> 0 -1 0
- joint waist_roll_joint: axis 1 0 0 -> -1 0 0; origin xyz=0.0039635 0 -0.044 rpy=0 0 0 -> xyz=0 0 0 rpy=0 0 0
- joint waist_yaw_joint: axis 0 0 1 -> 0 0 -1; origin xyz=0 0 0 rpy=0 0 0 -> xyz=0.0039635 0 -0.044 rpy=0 0 0
