Commit message: misc: b2 go2 newton mjwarp is checked, g1 is ongoing

File: source/locolab/locolab/assets/robots/unitree/G1/urdf/g1_description/g1_29dof_beyondmimic_pelvis_base.urdf (robot description, URDF)
Before this commit: robot g1, 40 links, 39 joints
Links:
- link left_hip_roll_link: geometry collision cylinder length=0.2 radius=0.051; visual mesh filename=meshes/left_hip_roll_link.STL
- link left_knee_link: geometry collision cylinder length=0.2 radius=0.052; visual mesh filename=meshes/left_knee_link.STL
- link right_hip_roll_link: geometry collision cylinder length=0.2 radius=0.051; visual mesh filename=meshes/right_hip_roll_link.STL
- link right_knee_link: geometry collision cylinder length=0.2 radius=0.052; visual mesh filename=meshes/right_knee_link.STL

File: source/locolab/locolab/assets/robots/unitree/G1/urdf/g1_description/g1_29dof_beyondmimic_torso_base.urdf (robot description, URDF)
Before this commit: robot g1, 40 links, 39 joints
Links:
- link left_hip_roll_link: geometry collision cylinder length=0.2 radius=0.051; visual mesh filename=meshes/left_hip_roll_link.STL
- link left_knee_link: geometry collision cylinder length=0.2 radius=0.052; visual mesh filename=meshes/left_knee_link.STL
- link right_hip_roll_link: geometry collision cylinder length=0.2 radius=0.051; visual mesh filename=meshes/right_hip_roll_link.STL
- link right_knee_link: geometry collision cylinder length=0.2 radius=0.052; visual mesh filename=meshes/right_knee_link.STL
