Commit message: update
1

stair still not good

615 test go2 env

File: source/locolab/locolab/assets/robots/unitree/Go2/urdf/go2_description/urdf/go2_description.urdf (robot description, URDF)
Before this commit: robot go2_description, 33 links, 32 joints
Links:
- link FL_calf: geometry collision box size=0.025 0.025 0.21; visual mesh filename=package://go2_description/dae/calf.dae
- link FL_thigh: geometry collision box size=0.20 0.0245 0.034; visual mesh filename=package://go2_description/dae/thigh.dae
- link FR_calf: geometry collision box size=0.025 0.025 0.21; visual mesh filename=package://go2_description/dae/calf_mirror.dae
- link FR_thigh: geometry collision box size=0.20 0.0245 0.034; visual mesh filename=package://go2_description/dae/thigh_mirror.dae
- link Head_upper: geometry collision box size=0.07 0.1 0.15
- link RL_calf: geometry collision box size=0.025 0.025 0.21; visual mesh filename=package://go2_description/dae/calf.dae
- link RL_thigh: geometry collision box size=0.20 0.0245 0.034; visual mesh filename=package://go2_description/dae/thigh.dae
- link RR_calf: geometry collision box size=0.025 0.025 0.21; visual mesh filename=package://go2_description/dae/calf_mirror.dae
- link RR_thigh: geometry collision box size=0.20 0.0245 0.034; visual mesh filename=package://go2_description/dae/thigh_mirror.dae
- link base: geometry collision box size=0.4 0.20 0.114; visual mesh filename=package://go2_description/dae/base.dae
