Commit message: update go2 asset

File: source/locolab/locolab/assets/robots/unitree/Go2/urdf/go2_description/urdf/go2_description_with_camera_30_bottom_collision.urdf (robot description, URDF)
Before this commit: robot go2_description, 33 links, 32 joints
Links:
- added link realsense_depth_origin_link, mass 0.072; visual sphere radius=0.003
- added link realsense_rack_link, mass 0.032; collision box size=0.03 0.13 0.02; collision box size=0.04 0.13 0.03
- link base: geometry collision box size=0.4 0.20 0.114; visual mesh filename=package://go2_description/dae/base.dae
Joints:
- added joint realsense_depth_origin_joint: type fixed, parent base, child realsense_depth_origin_link, origin xyz=0.335 0.015 0.088 rpy=0 0 0
- added joint realsense_rack_joint: type fixed, parent base, child realsense_rack_link, origin xyz=0.286 0 0.081 rpy=0 0 3.14159
