Commit message: update

File: source/locolab/locolab/assets/robots/unitree/B2/urdf/b2_description/urdf/b2z1_description.urdf (robot description, URDF)
Before this commit: robot b2_description, 37 links, 36 joints
Links:
- added link ee_gripper_link, mass 0.001
- added link gripperMover, mass 0.27621302; visual mesh filename=./meshes/z1_GripperMover.dae scale=1 1 1
- added link gripperStator, mass 0.52603655; collision box size=0.1 0.1 0.08; visual mesh filename=./meshes/z1_GripperStator.dae scale=1 1 1
- added link link00, mass 0.47247481; visual mesh filename=package://z1_description/meshes/visual/z1_Link00.dae scale=1 1 1
- added link link01, mass 0.67332551; visual mesh filename=package://z1_description/meshes/visual/z1_Link01.dae scale=1 1 1
- added link link02, mass 1.19132258; collision cylinder length=0.076 radius=0.0375; collision cylinder length=0.112 radius=0.0325
- added link link03, mass 0.83940874; collision cylinder length=0.072 radius=0.0325; collision cylinder length=0.116 radius=0.025
- added link link04, mass 0.56404563; visual mesh filename=package://z1_description/meshes/visual/z1_Link04.dae scale=1 1 1
- added link link05, mass 0.38938492; visual mesh filename=package://z1_description/meshes/visual/z1_Link05.dae scale=1 1 1
- added link link06, mass 0.28875807; collision cylinder length=0.051 radius=0.0375; visual mesh filename=package://z1_description/meshes/visual/z1_Link06.dae scale=1 1 1
- added link z1_arm_plat_link, mass 1.81613331316658; visual mesh filename=package://b2_description/meshes/z1_arm_plat_link.dae
Joints:
- added joint arm_plat_joint: type fixed, parent base_link, child z1_arm_plat_link, origin xyz=0.1745 0 0.088 rpy=0 0 0, axis 0 0 0
- added joint base_static_joint: type fixed, parent z1_arm_plat_link, child link00, origin xyz=0. 0. 0.173 rpy=0. 0. 0.
- added joint ee_gripper: type fixed, parent gripperStator, child ee_gripper_link, origin xyz=0.135 0 0 rpy=0 0 0, axis 1 0 0
- added joint gripperStator: type fixed, parent link06, child gripperStator, origin xyz=0.051 0.0 0.0 rpy=0 0 0
- added joint joint1: type revolute, parent link00, child link01, origin xyz=0 0 0.0585 rpy=0 0 0, axis 0 0 1, limit lower=-2.6179938779914944 upper=2.6179938779914944 effort=30.0 velocity=3.1415
- added joint joint2: type revolute, parent link01, child link02, origin xyz=0 0 0.045 rpy=0 0 0, axis 0 1 0, limit lower=0.0 upper=2.9670597283903604 effort=60.0 velocity=3.1415
- added joint joint3: type revolute, parent link02, child link03, origin xyz=-0.35 0 0 rpy=0 0 0, axis 0 1 0, limit lower=-2.8797932657906435 upper=0.0 effort=30.0 velocity=3.1415
- added joint joint4: type revolute, parent link03, child link04, origin xyz=0.218 0 0.057 rpy=0 0 0, axis 0 1 0, limit lower=-1.5184364492350666 upper=1.5184364492350666 effort=30.0 velocity=3.1415
- added joint joint5: type revolute, parent link04, child link05, origin xyz=0.07 0.0 0.0 rpy=0 0 0, axis 0 0 1, limit lower=-1.3439035240356338 upper=1.3439035240356338 effort=30.0 velocity=3.1415
- added joint joint6: type revolute, parent link05, child link06, origin xyz=0.0492 0.0 0.0 rpy=0 0 0, axis 1 0 0, limit lower=-2.792526803190927 upper=2.792526803190927 effort=30.0 velocity=3.1415
- added joint z1_jointGripper: type revolute, parent gripperStator, child gripperMover, origin xyz=0.049 0.0 0 rpy=0 0 0, axis 0 1 0, limit lower=-1.57 upper=0.0 effort=30.0 velocity=10

Commit message: update B2 assets

File: source/locolab/locolab/assets/robots/unitree/B2/urdf/b2_description/urdf/b2z1_description.urdf (robot description, URDF)
Before this commit: robot b2_description, 48 links, 47 joints
Joints:
- joint z1_jointGripper: type revolute -> fixed

Commit message: update b2z1 asset

File: source/locolab/locolab/assets/robots/unitree/B2/urdf/b2_description/urdf/b2z1_description.urdf (robot description, URDF)
Before this commit: robot b2_description, 48 links, 47 joints
Links:
- link base_link: geometry collision box size=0.14 0.24 0.19; collision box size=0.5 0.3 0.19
- link gripperMover: geometry visual mesh filename=package://b2_description/meshes/z1_GripperMover.dae scale=1 1 1
- link gripperStator: geometry collision box size=0.1 0.1 0.08; visual mesh filename=package://b2_description/meshes/z1_GripperStator.dae scale=1 1 1
- link link00: geometry visual mesh filename=package://b2_description/meshes/z1_Link00.dae scale=1 1 1
- link link01: geometry visual mesh filename=package://b2_description/meshes/z1_Link01.dae scale=1 1 1
- link link02: geometry collision cylinder length=0.4 radius=0.0225; visual mesh filename=package://b2_description/meshes/z1_Link02.dae scale=1 1 1
- link link03: geometry collision cylinder length=0.18 radius=0.025; visual mesh filename=package://b2_description/meshes/z1_Link03.dae scale=1 1 1
- link link04: geometry visual mesh filename=package://b2_description/meshes/z1_Link04.dae scale=1 1 1
- link link05: geometry visual mesh filename=package://b2_description/meshes/z1_Link05.dae scale=1 1 1
- link link06: geometry collision cylinder length=0.08 radius=0.0375; visual mesh filename=package://b2_description/meshes/z1_Link06.dae scale=1 1 1
- link z1_arm_plat_link: geometry visual mesh filename=package://b2_description/meshes/z1_arm_plat_link.stl
