Commit message: misc: archieve b2 go2 g1, use assetx for urdf/ujcf -> usd

File: source/locolab/locolab/assets/robots/unitree/B2/urdf/b2_description.urdf (robot description, URDF)
Before this commit: robot b2_description, 37 links, 36 joints
Links:
- link FL_calf: geometry collision box size=0.09 0.04 0.035; collision box size=0.3 0.045 0.03
- link FL_hip: geometry visual mesh filename=../meshes/FL_hip.dae
- link FL_thigh: geometry collision box size=0.40 0.05 0.06; visual mesh filename=../meshes/FL_thigh.dae
- link FR_calf: geometry collision box size=0.09 0.04 0.035; collision box size=0.3 0.045 0.03
- link FR_hip: geometry visual mesh filename=../meshes/FR_hip.dae
- link FR_thigh: geometry collision box size=0.40 0.05 0.06; visual mesh filename=../meshes/FR_thigh.dae
- link RL_calf: geometry collision box size=0.09 0.04 0.035; collision box size=0.3 0.045 0.03
- link RL_hip: geometry visual mesh filename=../meshes/RL_hip.dae
- link RL_thigh: geometry collision box size=0.40 0.05 0.06; visual mesh filename=../meshes/RL_thigh.dae
- link RR_calf: geometry collision box size=0.09 0.04 0.035; collision box size=0.3 0.045 0.03
- link RR_hip: geometry visual mesh filename=../meshes/RR_hip.dae
- link RR_thigh: geometry collision box size=0.40 0.05 0.06; visual mesh filename=../meshes/RR_thigh.dae
- link base_link: geometry collision box size=0.5 0.3 0.19; visual mesh filename=../meshes/base_link.dae

File: source/locolab/locolab/assets/robots/unitree/G1/urdf/g1_29dof_pelvis_base.urdf (robot description, URDF)
Before this commit: robot g1, 40 links, 39 joints
Links:
- link head_link: geometry visual mesh filename=../meshes/head_link.STL
- link left_ankle_pitch_link: geometry visual mesh filename=../meshes/left_ankle_pitch_link.STL
- link left_ankle_roll_link: geometry collision cylinder length=0.05 radius=0.01; collision cylinder length=0.05 radius=0.01
- link left_elbow_link: geometry collision cylinder length=0.13 radius=0.035; visual mesh filename=../meshes/left_elbow_link.STL
- link left_hip_pitch_link: geometry visual mesh filename=../meshes/left_hip_pitch_link.STL
- link left_hip_roll_link: geometry collision cylinder length=0.2 radius=0.051; visual mesh filename=../meshes/left_hip_roll_link.STL
- link left_hip_yaw_link: geometry visual mesh filename=../meshes/left_hip_yaw_link.STL
- link left_knee_link: geometry collision cylinder length=0.2 radius=0.052; visual mesh filename=../meshes/left_knee_link.STL
- link left_rubber_hand: geometry visual mesh filename=../meshes/left_rubber_hand.STL
- link left_shoulder_pitch_link: geometry visual mesh filename=../meshes/left_shoulder_pitch_link.STL
- link left_shoulder_roll_link: geometry visual mesh filename=../meshes/left_shoulder_roll_link.STL
- link left_shoulder_yaw_link: geometry collision cylinder length=0.13 radius=0.035; visual mesh filename=../meshes/left_shoulder_yaw_link.STL
- link left_wrist_pitch_link: geometry visual mesh filename=../meshes/left_wrist_pitch_link.STL
- link left_wrist_roll_link: geometry visual mesh filename=../meshes/left_wrist_roll_link.STL
- link left_wrist_yaw_link: geometry collision cylinder length=0.05 radius=0.05; visual mesh filename=../meshes/left_wrist_yaw_link.STL
- link logo_link: geometry visual mesh filename=../meshes/logo_link.STL
- link pelvis: geometry collision sphere radius=0.07; visual mesh filename=../meshes/pelvis.STL
- link pelvis_contour_link: geometry visual mesh filename=../meshes/pelvis_contour_link.STL
- link right_ankle_pitch_link: geometry visual mesh filename=../meshes/right_ankle_pitch_link.STL
- link right_ankle_roll_link: geometry collision cylinder length=0.05 radius=0.01; collision cylinder length=0.05 radius=0.01
- link right_elbow_link: geometry collision cylinder length=0.13 radius=0.035; visual mesh filename=../meshes/right_elbow_link.STL
- link right_hip_pitch_link: geometry visual mesh filename=../meshes/right_hip_pitch_link.STL
- link right_hip_roll_link: geometry collision cylinder length=0.2 radius=0.051; visual mesh filename=../meshes/right_hip_roll_link.STL
- link right_hip_yaw_link: geometry visual mesh filename=../meshes/right_hip_yaw_link.STL
- link right_knee_link: geometry collision cylinder length=0.2 radius=0.052; visual mesh filename=../meshes/right_knee_link.STL
- link right_rubber_hand: geometry visual mesh filename=../meshes/right_rubber_hand.STL
- link right_shoulder_pitch_link: geometry visual mesh filename=../meshes/right_shoulder_pitch_link.STL
- link right_shoulder_roll_link: geometry visual mesh filename=../meshes/right_shoulder_roll_link.STL
- link right_shoulder_yaw_link: geometry collision cylinder length=0.13 radius=0.035; visual mesh filename=../meshes/right_shoulder_yaw_link.STL
- link right_wrist_pitch_link: geometry visual mesh filename=../meshes/right_wrist_pitch_link.STL
- link right_wrist_roll_link: geometry visual mesh filename=../meshes/right_wrist_roll_link.STL
- link right_wrist_yaw_link: geometry collision cylinder length=0.05 radius=0.05; visual mesh filename=../meshes/right_wrist_yaw_link.STL
- link torso_link: geometry collision cylinder length=0.01 radius=0.068; collision cylinder length=0.04 radius=0.065
- link waist_roll_link: geometry visual mesh filename=../meshes/waist_roll_link_rev_1_0.STL
- link waist_yaw_link: geometry visual mesh filename=../meshes/waist_yaw_link_rev_1_0.STL
Joints:
- joint waist_pitch_joint: axis 0 -1 0 -> 0 1 0; child waist_roll_link -> torso_link; parent torso_link -> waist_roll_link
- joint waist_roll_joint: axis -1 0 0 -> 1 0 0; child waist_yaw_link -> waist_roll_link; origin xyz=0 0 0 rpy=0 0 0 -> xyz=-0.0039635 0 0.044 rpy=0 0 0; parent waist_roll_link -> waist_yaw_link
- joint waist_yaw_joint: axis 0 0 -1 -> 0 0 1; child pelvis -> waist_yaw_link; origin xyz=0.0039635 0 -0.044 rpy=0 0 0 -> xyz=0 0 0 rpy=0 0 0; parent waist_yaw_link -> pelvis

File: source/locolab/locolab/assets/robots/unitree/G1/urdf/g1_29dof_torso_base.urdf (robot description, URDF)
Before this commit: robot g1, 40 links, 39 joints
Links:
- link head_link: geometry visual mesh filename=../meshes/head_link.STL
- link left_ankle_pitch_link: geometry visual mesh filename=../meshes/left_ankle_pitch_link.STL
- link left_ankle_roll_link: geometry collision cylinder length=0.05 radius=0.01; collision cylinder length=0.05 radius=0.01
- link left_elbow_link: geometry collision cylinder length=0.13 radius=0.035; visual mesh filename=../meshes/left_elbow_link.STL
- link left_hip_pitch_link: geometry visual mesh filename=../meshes/left_hip_pitch_link.STL
- link left_hip_roll_link: geometry collision cylinder length=0.2 radius=0.051; visual mesh filename=../meshes/left_hip_roll_link.STL
- link left_hip_yaw_link: geometry visual mesh filename=../meshes/left_hip_yaw_link.STL
- link left_knee_link: geometry collision cylinder length=0.2 radius=0.052; visual mesh filename=../meshes/left_knee_link.STL
- link left_rubber_hand: geometry visual mesh filename=../meshes/left_rubber_hand.STL
- link left_shoulder_pitch_link: geometry visual mesh filename=../meshes/left_shoulder_pitch_link.STL
- link left_shoulder_roll_link: geometry visual mesh filename=../meshes/left_shoulder_roll_link.STL
- link left_shoulder_yaw_link: geometry collision cylinder length=0.13 radius=0.035; visual mesh filename=../meshes/left_shoulder_yaw_link.STL
- link left_wrist_pitch_link: geometry visual mesh filename=../meshes/left_wrist_pitch_link.STL
- link left_wrist_roll_link: geometry visual mesh filename=../meshes/left_wrist_roll_link.STL
- link left_wrist_yaw_link: geometry collision cylinder length=0.05 radius=0.05; visual mesh filename=../meshes/left_wrist_yaw_link.STL
- link logo_link: geometry visual mesh filename=../meshes/logo_link.STL
- link pelvis: geometry collision sphere radius=0.07; visual mesh filename=../meshes/pelvis.STL
- link pelvis_contour_link: geometry visual mesh filename=../meshes/pelvis_contour_link.STL
- link right_ankle_pitch_link: geometry visual mesh filename=../meshes/right_ankle_pitch_link.STL
- link right_ankle_roll_link: geometry collision cylinder length=0.05 radius=0.01; collision cylinder length=0.05 radius=0.01
- link right_elbow_link: geometry collision cylinder length=0.13 radius=0.035; visual mesh filename=../meshes/right_elbow_link.STL
- link right_hip_pitch_link: geometry visual mesh filename=../meshes/right_hip_pitch_link.STL
- link right_hip_roll_link: geometry collision cylinder length=0.2 radius=0.051; visual mesh filename=../meshes/right_hip_roll_link.STL
- link right_hip_yaw_link: geometry visual mesh filename=../meshes/right_hip_yaw_link.STL
- link right_knee_link: geometry collision cylinder length=0.2 radius=0.052; visual mesh filename=../meshes/right_knee_link.STL
- link right_rubber_hand: geometry visual mesh filename=../meshes/right_rubber_hand.STL
- link right_shoulder_pitch_link: geometry visual mesh filename=../meshes/right_shoulder_pitch_link.STL
- link right_shoulder_roll_link: geometry visual mesh filename=../meshes/right_shoulder_roll_link.STL
- link right_shoulder_yaw_link: geometry collision cylinder length=0.13 radius=0.035; visual mesh filename=../meshes/right_shoulder_yaw_link.STL
- link right_wrist_pitch_link: geometry visual mesh filename=../meshes/right_wrist_pitch_link.STL
- link right_wrist_roll_link: geometry visual mesh filename=../meshes/right_wrist_roll_link.STL
- link right_wrist_yaw_link: geometry collision cylinder length=0.05 radius=0.05; visual mesh filename=../meshes/right_wrist_yaw_link.STL
- link torso_link: geometry collision cylinder length=0.01 radius=0.068; collision cylinder length=0.04 radius=0.065
- link waist_roll_link: geometry visual mesh filename=../meshes/waist_roll_link_rev_1_0.STL
- link waist_yaw_link: geometry visual mesh filename=../meshes/waist_yaw_link_rev_1_0.STL
Joints:
- joint waist_pitch_joint: axis 0 1 0 -> 0 -1 0; child torso_link -> waist_roll_link; parent waist_roll_link -> torso_link
- joint waist_roll_joint: axis 1 0 0 -> -1 0 0; child waist_roll_link -> waist_yaw_link; origin xyz=-0.0039635 0 0.044 rpy=0 0 0 -> xyz=0 0 0 rpy=0 0 0; parent waist_yaw_link -> waist_roll_link
- joint waist_yaw_joint: axis 0 0 1 -> 0 0 -1; child waist_yaw_link -> pelvis; origin xyz=0 0 0 rpy=0 0 0 -> xyz=0.0039635 0 -0.044 rpy=0 0 0; parent pelvis -> waist_yaw_link

File: source/locolab/locolab/assets/robots/unitree/Go2/urdf/go2_description.urdf (robot description, URDF)
Before this commit: robot go2_description, 33 links, 32 joints
Links:
- link FL_calf: geometry collision box size=0.025 0.025 0.21; visual mesh filename=../meshes/calf.dae
- link FL_foot: geometry collision sphere radius=0.022; visual mesh filename=../meshes/foot.dae
- link FL_hip: geometry visual mesh filename=../meshes/hip.dae
- link FL_thigh: geometry collision box size=0.20 0.0245 0.034; visual mesh filename=../meshes/thigh.dae
- link FR_calf: geometry collision box size=0.025 0.025 0.21; visual mesh filename=../meshes/calf_mirror.dae
- link FR_foot: geometry collision sphere radius=0.022; visual mesh filename=../meshes/foot.dae
- link FR_hip: geometry visual mesh filename=../meshes/hip.dae
- link FR_thigh: geometry collision box size=0.20 0.0245 0.034; visual mesh filename=../meshes/thigh_mirror.dae
- link RL_calf: geometry collision box size=0.025 0.025 0.21; visual mesh filename=../meshes/calf.dae
- link RL_foot: geometry collision sphere radius=0.022; visual mesh filename=../meshes/foot.dae
- link RL_hip: geometry visual mesh filename=../meshes/hip.dae
- link RL_thigh: geometry collision box size=0.20 0.0245 0.034; visual mesh filename=../meshes/thigh.dae
- link RR_calf: geometry collision box size=0.025 0.025 0.21; visual mesh filename=../meshes/calf_mirror.dae
- link RR_foot: geometry collision sphere radius=0.022; visual mesh filename=../meshes/foot.dae
- link RR_hip: geometry visual mesh filename=../meshes/hip.dae
- link RR_thigh: geometry collision box size=0.20 0.0245 0.034; visual mesh filename=../meshes/thigh_mirror.dae
- link base: geometry collision box size=0.07 0.10 0.13; collision box size=0.4 0.20 0.12
